File: kicad/split_keyboard/split_keyboard.kicad_pcb (KiCad board)
At the start: 2 copper layers, 180.3 x 134.6 mm, 79 parts, among them J1 Conn_02x08_Odd_Even, SW1 SW_PUSH, SW10 SW_PUSH, SW11 SW_PUSH, SW12 SW_PUSH, SW13 SW_PUSH, SW14 SW_PUSH, SW15 SW_PUSH, SW16 SW_PUSH, SW17 SW_PUSH, SW18 SW_PUSH, SW19 SW_PUSH, SW2 SW_PUSH, SW20 SW_PUSH, SW21 SW_PUSH, SW22 SW_PUSH, SW23 SW_PUSH, SW24 SW_PUSH, SW25 SW_PUSH, SW26 SW_PUSH, SW27 SW_PUSH, SW28 SW_PUSH, SW29 SW_PUSH, SW3 SW_PUSH, SW30 SW_PUSH, SW31 SW_PUSH, SW32 SW_PUSH, SW33 SW_PUSH, SW34 SW_PUSH, SW35 SW_PUSH, SW36 SW_PUSH, SW4 SW_PUSH, SW5 SW_PUSH, SW6 SW_PUSH, SW7 SW_PUSH, SW8 SW_PUSH, SW9 SW_PUSH, U1 ESP32-DEVKITC-32D

Commit message: complete lefthand pcb.
Parts:
- added R1: R, Resistor_THT:R_Axial_DIN0204_L3.6mm_D1.6mm_P2.54mm_Vertical, F.Cu at (194.3, 63.5)
- added R2: R, Resistor_THT:R_Axial_DIN0204_L3.6mm_D1.6mm_P2.54mm_Vertical, F.Cu at (194.3, 66.0)
- added R3: R, Resistor_THT:R_Axial_DIN0204_L3.6mm_D1.6mm_P2.54mm_Vertical, F.Cu at (194.3, 68.6)
- added R4: R, Resistor_THT:R_Axial_DIN0204_L3.6mm_D1.6mm_P2.54mm_Vertical, F.Cu at (194.3, 71.1)
- moved D1 2.54 mm to (38.7, 46.4)
- moved D10 2.54 mm to (76.8, 65.4)
- moved D13 2.54 mm to (95.9, 46.4)
- moved D14 2.54 mm to (95.9, 65.4)
- moved D17 2.54 mm to (114.9, 46.4)
- moved D18 2.54 mm to (114.9, 65.4)
- moved D2 2.54 mm to (38.7, 65.4)
- moved D21 2.54 mm to (134.0, 46.4)
- moved D22 2.54 mm to (134.0, 65.4)
- moved D3 2.54 mm to (57.8, 46.4)
- moved D4 2.54 mm to (57.8, 65.4)
- moved D9 2.54 mm to (76.8, 46.4)
- moved D11 2.54 mm to (86.4, 84.5)
- moved D12 2.54 mm to (90.8, 103.5)
- moved D15 2.54 mm to (105.4, 84.5)
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Routing:
- net ROW_2: track 223.8 -> 311.3 mm, vias 0 -> 4
- net ROW_1: track 253.8 -> 332.6 mm
- net COL_6: track 302.8 -> 244.7 mm, vias 0 -> 1
- net +5V: track 0.00 -> 53.4 mm
- net VCC: track 51.9 -> 68.5 mm, vias 0 -> 1
- net ROW_0: track 412.4 -> 420.2 mm
- net COL_8: track 208.1 -> 202.3 mm
- net COL_2: track 264.9 -> 269.9 mm, vias 0 -> 1
- net ROW_3: track 265.5 -> 270.1 mm
- net Net-(D9-Pad2): track 15.8 -> 19.6 mm
- net COL_7: track 231.7 -> 228.5 mm
- net Net-(D6-Pad2): track 15.6 -> 18.8 mm
- net Net-(D24-Pad2): track 14.8 -> 18.0 mm
- net Net-(D20-Pad2): track 14.8 -> 18.0 mm
- net Net-(D11-Pad2): track 15.8 -> 18.9 mm
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- added copper zone on B.Cu, net GND
- added copper zone on F.Cu, net GND

Commit message: complete to design pcb, and export gerber data.
Parts:
- added C1: CP, Capacitor_THT:CP_Radial_D5.0mm_P2.50mm, F.Cu at (177.8, 133.3)
- added J2: Conn_01x04, Connector_PinSocket_2.54mm:PinSocket_1x04_P2.54mm_Vertical, F.Cu at (180.3, 127.0)
- added J3: Conn_01x04, Connector_PinSocket_2.54mm:PinSocket_1x04_P2.54mm_Vertical, F.Cu at (172.7, 127.0)
- R1, R2, R3, R4: footprint Resistor_THT:R_Axial_DIN0204_L3.6mm_D1.6mm_P2.54mm_Vertical -> Resistor_THT:R_Axial_DIN0207_L6.3mm_D2.5mm_P2.54mm_Vertical
- U1: footprint MODULE_ESP32-DEVKITC-32D -> ESP32-DEVKITC-32D:MODULE_ESP32-DEVKITC-32D
- moved D28 1.91 mm to (156.2, 120.0)
- moved R1 1.27 mm to (194.3, 62.2)
- moved R2 0.64 mm to (194.3, 65.4)
- moved R4 0.63 mm to (194.3, 71.8)
Connections:
- U1 pad 14: +5V -> GND
- U1 pad 20: +5V -> GND
- U1 pad 26: +5V -> GND
Routing:
- net GND: track 0.00 -> 53.4 mm, vias 99 -> 97
- net +5V: track 53.4 -> 0.00 mm
- net VCC: track 68.5 -> 97.3 mm
- net ROW_3: track 270.1 -> 267.8 mm
- net Net-(D28-Pad2): vias 1 -> 0
