File: kicad/split_keyboard_righthand/split_keyboard_righthand.kicad_pcb (KiCad board)
At the start: 2 copper layers, 188.1 x 133.3 mm, 99 parts, among them J1 Conn_02x08_Odd_Even, SW1 SW_PUSH, SW10 SW_PUSH, SW11 SW_PUSH, SW12 SW_PUSH, SW13 SW_PUSH, SW14 SW_PUSH, SW15 SW_PUSH, SW16 SW_PUSH, SW17 SW_PUSH, SW18 SW_PUSH, SW19 SW_PUSH, SW2 SW_PUSH, SW20 SW_PUSH, SW21 SW_PUSH, SW22 SW_PUSH, SW23 SW_PUSH, SW24 SW_PUSH, SW25 SW_PUSH, SW26 SW_PUSH, SW27 SW_PUSH, SW28 SW_PUSH, SW29 SW_PUSH, SW3 SW_PUSH, SW30 SW_PUSH, SW31 SW_PUSH, SW32 SW_PUSH, SW33 SW_PUSH, SW34 SW_PUSH, SW35 SW_PUSH, SW36 SW_PUSH, SW37 SW_PUSH, SW38 SW_PUSH, SW39 SW_PUSH, SW4 SW_PUSH, SW40 SW_PUSH, SW41 SW_PUSH, SW42 SW_PUSH, SW43 SW_PUSH, SW44 SW_PUSH, SW45 SW_PUSH, SW5 SW_PUSH, SW6 SW_PUSH, SW7 SW_PUSH, SW8 SW_PUSH, SW9 SW_PUSH

Commit message: complete lefthand pcb.
Parts:
- C1: footprint Capacitor_THT:CP_Radial_D5.0mm_P2.50mm -> Capacitor_THT:C_Disc_D3.0mm_W1.6mm_P2.50mm
- D46: footprint LED_THT:LED_D1.8mm_W1.8mm_H2.4mm_Horizontal_O3.81mm_Z1.6mm -> LED_THT:LED_D3.0mm_FlatTop
- R1: value R -> R_Axial_DIN0207_L6.3mm_D2.5mm_P10.16mm_Horizontal; footprint kbd:R -> Resistor_THT:R_Axial_DIN0207_L6.3mm_D2.5mm_P10.16mm_Horizontal
- moved C1 14.2 mm to (31.8, 91.4)
- moved R1 10.5 mm to (29.2, 83.8), turned to 270 degrees
- moved D46 9.49 mm to (29.2, 99.1)
Routing:
- net GND: track 0.00 -> 72.5 mm
- net VCC: track 0.00 -> 31.7 mm
- net Net-(D46-Pad1): track 0.00 -> 5.08 mm

Commit message: complete to design pcb, and export gerber data.
Parts:
- C1: footprint Capacitor_THT:C_Disc_D3.0mm_W1.6mm_P2.50mm -> Capacitor_THT:CP_Radial_D5.0mm_P2.50mm
- R1: value R_Axial_DIN0207_L6.3mm_D2.5mm_P10.16mm_Horizontal -> R; footprint Resistor_THT:R_Axial_DIN0207_L6.3mm_D2.5mm_P10.16mm_Horizontal -> Resistor_THT:R_Axial_DIN0207_L6.3mm_D2.5mm_P7.62mm_Horizontal
- moved D46 1.27 mm to (27.9, 99.1)
- moved R1 1.27 mm to (27.9, 83.8)
Routing:
- net GND: track 72.5 -> 78.2 mm
- net ROW_6: track 259.8 -> 263.1 mm
- net Net-(D46-Pad1): track 5.08 -> 7.62 mm
- net VCC: track 31.7 -> 32.8 mm
- net COL_7: track 361.5 -> 362.0 mm
- added copper zone on B.Cu, net GND
- added copper zone on F.Cu, net GND
