File: kicad/skb_i2c_lefthand/file6006EC2F.sch (KiCad schematic (older format))
At the start: 80 parts, among them SW1 SW_PUSH, SW10 SW_PUSH, SW11 SW_PUSH, SW12 SW_PUSH, SW13 SW_PUSH, SW14 SW_PUSH, SW17 SW_PUSH, SW18 SW_PUSH, SW19 SW_PUSH, SW2 SW_PUSH, SW20 SW_PUSH, SW21 SW_PUSH, SW22 SW_PUSH, SW23 SW_PUSH, SW25 SW_PUSH, SW26 SW_PUSH, SW27 SW_PUSH, SW28 SW_PUSH, SW29 SW_PUSH, SW3 SW_PUSH, SW30 SW_PUSH, SW31 SW_PUSH, SW33 SW_PUSH, SW34 SW_PUSH, SW35 SW_PUSH, SW36 SW_PUSH, SW37 SW_PUSH, SW38 SW_PUSH, SW39 SW_PUSH, SW4 SW_PUSH, SW41 SW_PUSH, SW42 SW_PUSH, SW43 SW_PUSH, SW44 SW_PUSH, SW45 SW_PUSH, SW46 SW_PUSH, SW47 SW_PUSH, SW5 SW_PUSH, SW6 SW_PUSH, SW9 SW_PUSH

Commit message: route roughly
Parts:
- removed D23, D31, D39, D47: 1N4148, Diode_THT:D_DO-35_SOD27_P7.62mm_Horizontal, symbol Diode:1N4148
- removed SW23, SW31, SW39, SW47: SW_PUSH, kbd:CherryMX_1u, symbol kbd:SW_PUSH
- SW1, SW10, SW11, SW12, SW13, SW14, SW17, SW18, SW19, SW2, SW20, SW21, SW22, SW25, SW26, SW27, SW28, SW29, SW3, SW30, SW33, SW34, SW35, SW36, SW37, SW38, SW4, SW41, SW42, SW43, SW44, SW45, SW46, SW5, SW6, SW9: footprint kbd:CherryMX_1u -> keyboard_parts:Kailh_MX_Socket
Connections:
- wire segments 101 -> 89
