File: kicad/skb_i2c_lefthand/skb_i2c_lefthand.kicad_pcb (KiCad board)
At the start: 2 copper layers, 96 parts, among them J1 Conn_01x05_Male, J3 Power, J4 Conn_01x04_Male, J5 Conn_01x04_Male, J6 MJ-4PP-9, SW1 SW_PUSH, SW10 SW_PUSH, SW11 SW_PUSH, SW12 SW_PUSH, SW13 SW_PUSH, SW14 SW_PUSH, SW17 SW_PUSH, SW18 SW_PUSH, SW19 SW_PUSH, SW2 SW_PUSH, SW20 SW_PUSH, SW21 SW_PUSH, SW22 SW_PUSH, SW23 SW_PUSH, SW25 SW_PUSH, SW26 SW_PUSH, SW27 SW_PUSH, SW28 SW_PUSH, SW29 SW_PUSH, SW3 SW_PUSH, SW30 SW_PUSH, SW31 SW_PUSH, SW33 SW_PUSH, SW34 SW_PUSH, SW35 SW_PUSH, SW36 SW_PUSH, SW37 SW_PUSH, SW38 SW_PUSH, SW39 SW_PUSH, SW4 SW_PUSH, SW41 SW_PUSH, SW42 SW_PUSH, SW43 SW_PUSH, SW44 SW_PUSH, SW45 SW_PUSH, SW46 SW_PUSH, SW47 SW_PUSH, SW5 SW_PUSH, SW6 SW_PUSH, SW9 SW_PUSH, U1 MCP23017_SO, U2 PCA9515AD

Commit message: route roughly
Parts:
- removed D23, D31, D39, D47: 1N4148, Diode_THT:D_DO-35_SOD27_P7.62mm_Horizontal
- removed SW23, SW31, SW39, SW47: SW_PUSH, kbd:CherryMX_1u
- added Ref**: Val**, kbd:HOLE, F.Cu at (90.8, 135.9)
- added Ref**: Val**, kbd:HOLE, F.Cu at (142.2, 42.5)
- added Ref**: Val**, kbd:HOLE, F.Cu at (31.1, 44.5)
- added Ref**: Val**, kbd:HOLE, F.Cu at (31.8, 139.7)
- added Ref**: Val**, kbd:HOLE, F.Cu at (163.2, 139.7)
- C1: footprint Capacitor_THT:CP_Axial_L10.0mm_D4.5mm_P15.00mm_Horizontal -> Capacitor_THT:CP_Radial_D5.0mm_P2.50mm
- J1, J3, J4, J5, J6, JP1, JP2, JP3, R1, R2: moved to B.Cu
- JP4: value SCL -> I2C_SCL; footprint Jumper:SolderJumper-2_P1.3mm_Open_RoundedPad1.0x1.5mm -> Jumper:SolderJumper-3_P1.3mm_Open_RoundedPad1.0x1.5mm
- JP5: value SDA -> I2C_SDA; footprint Jumper:SolderJumper-2_P1.3mm_Open_RoundedPad1.0x1.5mm -> Jumper:SolderJumper-3_P1.3mm_Open_RoundedPad1.0x1.5mm
- SW1, SW10, SW11, SW12, SW13, SW14, SW17, SW18, SW19, SW2, SW20, SW21, SW22, SW25, SW26, SW27, SW28, SW29, SW3, SW30, SW33, SW34, SW35, SW36, SW37, SW38, SW4, SW41, SW42, SW43, SW44, SW45, SW46, SW5, SW6, SW9: footprint kbd:CherryMX_1u -> keyboard_parts:Kailh_MX_Socket
- moved JP1 162.7 mm to (50.8, 128.3), turned to 180 degrees
- moved JP3 160.8 mm to (55.9, 123.2), turned to 180 degrees
- moved JP2 153.7 mm to (50.8, 125.7), turned to 180 degrees
- moved JP6 127.8 mm to (31.8, 124.0)
- moved JP4 119.2 mm to (35.6, 112.8)
- moved U2 118.2 mm to (35.6, 116.8)
- moved JP5 117.7 mm to (35.6, 121.4)
- moved R1 116.1 mm to (80.0, 124.5)
- moved R2 108.7 mm to (80.0, 121.9)
- moved C1 103.7 mm to (59.1, 100.3), turned to 270 degrees
- moved J1 78.1 mm to (104.1, 42.5)
- moved J6 76.8 mm to (125.1, 27.9), turned to 180 degrees
- moved J3 69.3 mm to (55.9, 90.2), turned to 180 degrees
- moved J4 60.9 mm to (116.8, 41.9)
- moved J5 50.3 mm to (85.1, 40.0)
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Connections:
- JP1 pad 1: +5V -> GND
- JP1 pad 3: VCC -> VCC5V
- JP2 pad 1: +5V -> GND
- JP2 pad 3: VCC -> VCC5V
- JP3 pad 1: +5V -> GND
- JP3 pad 3: VCC -> VCC5V
- JP6 pad 2: VCC -> VCC5V
- R1 pad 1: VCC -> VCC5V
- R2 pad 1: VCC -> VCC5V
- U1 pad 10: +5V -> GND
- U1 pad 18: VCC -> VCC5V
- U1 pad 9: VCC -> VCC5V
- U2 pad 4: +5V -> GND
- U2 pad 6: SDA_MCP -> Net-(JP5-Pad3)
- U2 pad 7: SCL_MCP -> Net-(JP4-Pad3)
- U2 pad 8: VCC -> VCC5V
Routing:
- net GND: track 0.00 -> 353.4 mm, vias 0 -> 10
- net VCC5V: track 0.00 -> 268.6 mm, vias 0 -> 7
- net COL_5: track 0.00 -> 201.5 mm, vias 0 -> 2
- net COL_4: track 0.00 -> 191.4 mm, vias 0 -> 2
- net SDA_GROVE: track 0.00 -> 185.7 mm, vias 0 -> 3
- net G33: track 163.5 -> 0.00 mm, vias 1 -> 0
- net VCC3P3V: track 0.00 -> 121.1 mm, vias 0 -> 1
- net COL_0: track 226.8 -> 128.9 mm, vias 1 -> 2
- net COL_1: track 217.7 -> 146.0 mm, vias 1 -> 4
- net ROW_0: track 129.5 -> 189.8 mm, vias 0 -> 1
- net COL_2: track 205.4 -> 157.2 mm, vias 1 -> 2
- net SCL_MCP: track 0.00 -> 44.9 mm, vias 0 -> 2
- net SDA_MCP: track 0.00 -> 43.4 mm, vias 0 -> 1
- net ROW_1: track 133.3 -> 168.5 mm, vias 0 -> 1
- net SCL_GROVE: track 135.3 -> 168.5 mm, vias 1 -> 3
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- added copper zone on B.Cu, net GND
- added copper zone on F.Cu, net GND
- added copper zone on F.Cu, net VCC5V
Other:
- board outline added: 139.1 x 115.6 mm
- net class POWER added: clearance 0.2, trace_width 0.5, via_dia 0.8, via_drill 0.4
