File: kicad/skb_i2c_righthand/skb_i2c_righthand.kicad_pcb (KiCad board)
At the start: 2 copper layers, 124 parts, among them J2_TRRS1 MJ-4PP-9, J3_PIKO_L1 Conn_01x05_Male, J3_PIKO_R1 Conn_01x04_Male, J4_GROVE1 Conn_01x04_Male, J5 Conn_01x04, SW1 SW_PUSH, SW10 SW_PUSH, SW11 SW_PUSH, SW12 SW_PUSH, SW13 SW_PUSH, SW14 SW_PUSH, SW15 SW_PUSH, SW16 SW_PUSH, SW17 SW_PUSH, SW18 SW_PUSH, SW19 SW_PUSH, SW2 SW_PUSH, SW20 SW_PUSH, SW21 SW_PUSH, SW22 SW_PUSH, SW23 SW_PUSH, SW24 SW_PUSH, SW25 SW_PUSH, SW26 SW_PUSH, SW27 SW_PUSH, SW28 SW_PUSH, SW29 SW_PUSH, SW3 SW_PUSH, SW30 SW_PUSH, SW31 SW_PUSH, SW32 SW_PUSH, SW33 SW_PUSH, SW34 SW_PUSH, SW35 SW_PUSH, SW36 SW_PUSH, SW37 SW_PUSH, SW38 SW_PUSH, SW39 SW_PUSH, SW4 SW_PUSH, SW40 SW_PUSH, SW41 SW_PUSH, SW42 SW_PUSH, SW43 SW_PUSH, SW44 SW_PUSH, SW45 SW_PUSH, SW46 SW_PUSH, SW47 SW_PUSH, SW48 SW_PUSH, SW49 SW_PUSH, SW5 SW_PUSH, SW50 SW_PUSH, SW51 SW_PUSH, SW52 SW_PUSH, SW53 SW_PUSH, SW54 SW_PUSH, SW6 SW_PUSH, SW7 SW_PUSH, SW8 SW_PUSH, SW9 SW_PUSH, U1 MCP23017_SO, U2 PCA9515AD

Commit message: route roughly
Parts:
- removed D46, D47, D48, D51, D52, D53, D54: 1N4148, Diode_THT:D_DO-35_SOD27_P7.62mm_Horizontal
- removed SW46, SW47, SW48, SW51, SW52, SW53, SW54: SW_PUSH, keyboard_parts:Kailh_MX_Socket
- C1: footprint Capacitor_THT:CP_Axial_L10.0mm_D4.5mm_P15.00mm_Horizontal -> Capacitor_THT:CP_Radial_D5.0mm_P2.50mm
- J2_TRRS1, J3_PIKO_L1, J3_PIKO_R1, J5, JP_A0, JP_A1, JP_A2, JP_I2C_EN1, U1, U2: moved to B.Cu
- JP_SCL1: value SCL -> I2C_A2; footprint Jumper:SolderJumper-2_P1.3mm_Open_RoundedPad1.0x1.5mm -> Jumper:SolderJumper-3_P1.3mm_Open_RoundedPad1.0x1.5mm_NumberLabels; moved to B.Cu
- JP_SDA1: value SDA -> I2C_A2; footprint Jumper:SolderJumper-2_P1.3mm_Open_RoundedPad1.0x1.5mm -> Jumper:SolderJumper-3_P1.3mm_Open_RoundedPad1.0x1.5mm_NumberLabels; moved to B.Cu
- moved R2 253.2 mm to (180.3, 91.4), turned to 90 degrees
- moved C1 247.2 mm to (175.3, 114.3), turned to 90 degrees
- moved R1 245.0 mm to (182.9, 91.4), turned to 90 degrees
- moved J5 238.2 mm to (180.3, 106.7), turned to 180 degrees
- moved JP_A0 230.4 mm to (188.0, 101.0), turned to 180 degrees
- moved JP_A1 223.9 mm to (188.0, 97.2), turned to 180 degrees
- moved JP_A2 222.3 mm to (188.0, 94.0), turned to 180 degrees
- moved U1 215.7 mm to (196.8, 91.4), turned to 180 degrees
- moved U2 214.5 mm to (180.3, 76.8)
- moved JP_SCL1 206.8 mm to (180.3, 81.3)
- moved JP_SDA1 201.6 mm to (179.7, 72.4)
- moved JP_I2C_EN1 199.8 mm to (179.1, 69.2), turned to 180 degrees
- moved J4_GROVE1 96.9 mm to (64.5, 36.8), turned to 270 degrees
- moved J3_PIKO_L1 63.9 mm to (91.4, 26.7), turned to 180 degrees
- moved J3_PIKO_R1 31.8 mm to (71.1, 26.7), turned to 180 degrees
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Connections:
- net ROW_6 renamed Net-(U1-Pad7)
- JP_A0 pad 1: +5V -> GND
- JP_A0 pad 3: VCC -> VCC5V
- JP_A1 pad 1: +5V -> GND
- JP_A1 pad 3: VCC -> VCC5V
- JP_A2 pad 1: +5V -> GND
- JP_A2 pad 3: VCC -> VCC5V
- JP_I2C_EN1 pad 2: VCC -> VCC5V
- R1 pad 1: VCC -> VCC5V
- R2 pad 1: VCC -> VCC5V
- U1 pad 10: +5V -> GND
- U1 pad 18: VCC -> VCC5V
- U1 pad 8: ROW_7 -> COL_8
- U1 pad 9: VCC -> VCC5V
- U2 pad 4: +5V -> GND
- U2 pad 6: SDA_MCP -> Net-(JP_SDA1-Pad3)
- U2 pad 7: SCL_MCP -> Net-(JP_SCL1-Pad3)
- U2 pad 8: VCC -> VCC5V
Routing:
- net VCC5V: track 0.00 -> 404.6 mm, vias 0 -> 4
- net GND: track 0.00 -> 383.9 mm, vias 0 -> 8
- net COL_0: track 0.00 -> 252.6 mm, vias 0 -> 2
- net COL_1: track 0.00 -> 243.2 mm, vias 0 -> 2
- net COL_2: track 0.00 -> 229.0 mm, vias 0 -> 2
- net ROW_0: track 0.00 -> 223.4 mm
- net COL_3: track 0.00 -> 208.9 mm, vias 0 -> 2
- net ROW_1: track 0.00 -> 207.6 mm
- net ROW_5: track 0.00 -> 193.2 mm, vias 0 -> 3
- net COL_4: track 0.00 -> 187.7 mm, vias 0 -> 2
- net SDA_GROVE: track 0.00 -> 182.2 mm, vias 0 -> 1
- net ROW_4: track 0.00 -> 181.8 mm, vias 0 -> 3
- net ROW_3: track 0.00 -> 176.8 mm, vias 0 -> 1
- net ROW_2: track 0.00 -> 174.2 mm
- net SCL_GROVE: track 0.00 -> 172.8 mm, vias 0 -> 1
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Other:
- net class POWER added: clearance 0.2, trace_width 0.5, via_dia 0.8, via_drill 0.4
