File: kicad/skb_i2c_twohand/file5FDF19E5.sch (KiCad schematic (older format))
At the start: 29 parts, among them J2_TRRS1 MJ-4PP-9, J3_PIKO_L1 Conn_01x05_Male, J3_PIKO_R1 Conn_01x04_Male, J4_GROVE1 Conn_01x04_Male, J6 Conn_01x04, SW85 SW_DIP_x01, U3 MCP23017_SO, U4 PCA9515AD

Commit message: route
Parts:
- added J10, J9: Conn_01x03, Connector_PinHeader_2.54mm:PinHeader_1x03_P2.54mm_Vertical, symbol Connector_Generic:Conn_01x03
Connections:
- net G22: now also J9.1 (Pin_1), J9.2 (Pin_2), J9.3 (Pin_3)
- net G33: now also J10.1 (Pin_1), J10.2 (Pin_2), J10.3 (Pin_3)
- net VCC3P3V: now also SW85.1; no longer C2.1, J6.4 (Pin_4)
- net VCC5V: now also JP_A1.3 (B), JP_A2.3 (B), JP_A3.3 (B); no longer SW85.2
- removed net VCC: JP_A1.3 (B), JP_A2.3 (B), JP_A3.3 (B), SW85.1
- new net VCC3P3V_T: C2.1, J6.4 (Pin_4), SW85.2
- no-connect marks 10 -> 8
Other:
- note removed: "M5 ATOM"
- moved on the sheet: J3_PIKO_L1, J3_PIKO_R1, SW85
