File: kicad/skb_i2c_twohand/skb_i2c_lefthand.kicad_pcb (KiCad board)
At the start: 2 copper layers, 353.7 x 115.6 mm, 212 parts, among them J1 MJ-4PP-9, J2 Conn_01x05_Male, J2_TRRS1 MJ-4PP-9, J3 Conn_01x04_Male, J3_PIKO_L1 Conn_01x05_Male, J3_PIKO_R1 Conn_01x04_Male, J4 Power, J4_GROVE1 Conn_01x04_Male, J5 Conn_01x04_Male, J6 Conn_01x04, SW1 SW_PUSH, SW10 SW_PUSH, SW11 SW_PUSH, SW12 SW_PUSH, SW13 SW_PUSH, SW14 SW_PUSH, SW15 SW_PUSH, SW16 SW_PUSH, SW17 SW_PUSH, SW18 SW_PUSH, SW19 SW_PUSH, SW2 SW_PUSH, SW20 SW_PUSH, SW21 SW_PUSH, SW22 SW_PUSH, SW23 SW_PUSH, SW24 SW_PUSH, SW25 SW_PUSH, SW26 SW_PUSH, SW27 SW_PUSH, SW28 SW_PUSH, SW29 SW_PUSH, SW3 SW_PUSH, SW30 SW_PUSH, SW31 SW_PUSH, SW32 SW_PUSH, SW33 SW_PUSH, SW34 SW_PUSH, SW35 SW_PUSH, SW36 SW_PUSH, SW37 SW_PUSH, SW38 SW_PUSH, SW39 SW_PUSH, SW4 SW_PUSH, SW40 SW_PUSH, SW41 SW_PUSH, SW42 SW_PUSH, SW43 SW_PUSH, SW44 SW_PUSH, SW45 SW_PUSH, SW46 SW_PUSH, SW47 SW_PUSH, SW48 SW_PUSH, SW49 SW_PUSH, SW5 SW_PUSH, SW50 SW_PUSH, SW51 SW_PUSH, SW52 SW_PUSH, SW53 SW_PUSH, SW54 SW_PUSH, SW55 SW_PUSH, SW56 SW_PUSH, SW57 SW_PUSH, SW58 SW_PUSH, SW59 SW_PUSH, SW6 SW_PUSH, SW60 SW_PUSH, SW61 SW_PUSH, SW62 SW_PUSH, SW63 SW_PUSH, SW64 SW_PUSH, SW65 SW_PUSH, SW66 SW_PUSH, SW67 SW_PUSH, SW68 SW_PUSH, SW69 SW_PUSH, SW7 SW_PUSH, SW70 SW_PUSH, SW71 SW_PUSH, SW72 SW_PUSH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

Commit message: route
Parts:
- added D84: LED, LED_THT:LED_D3.0mm, F.Cu at (168.1, 141.2)
- added D85: LED, LED_THT:LED_D3.0mm, F.Cu at (146.8, 30.5)
- added J10: Conn_01x03, Connector_PinHeader_2.54mm:PinHeader_1x03_P2.54mm_Vertical, F.Cu at (177.0, 39.6)
- added J7: Conn_01x03, Connector_PinHeader_2.54mm:PinHeader_1x03_P2.54mm_Vertical, F.Cu at (170.7, 137.2)
- added J8: Conn_01x03, Connector_PinHeader_2.54mm:PinHeader_1x03_P2.54mm_Vertical, F.Cu at (149.4, 39.6)
- added J9: Conn_01x03, Connector_PinHeader_2.54mm:PinHeader_1x03_P2.54mm_Vertical, F.Cu at (198.4, 137.2)
- added R5: R, Resistor_THT:R_Axial_DIN0204_L3.6mm_D1.6mm_P7.62mm_Horizontal, F.Cu at (167.6, 130.0)
- added R6: R, Resistor_THT:R_Axial_DIN0204_L3.6mm_D1.6mm_P7.62mm_Horizontal, F.Cu at (146.3, 41.4)
- added Ref**: Val**, kbd:HOLE, F.Cu at (278.6, 137.4)
- added Ref**: Val**, kbd:HOLE, F.Cu at (204.2, 139.4)
- added Ref**: Val**, kbd:HOLE, F.Cu at (161.8, 139.4)
- added Ref**: Val**, kbd:HOLE, F.Cu at (279.4, 31.0)
- added Ref**: Val**, kbd:HOLE, F.Cu at (90.9, 137.4)
- added Ref**: Val**, kbd:HOLE, F.Cu at (32.0, 44.2)
- added Ref**: Val**, kbd:HOLE, F.Cu at (145.3, 47.5)
- added Ref**: Val**, kbd:HOLE, F.Cu at (350.0, 137.9)
- added Ref**: Val**, kbd:HOLE, F.Cu at (179.1, 47.5)
- added Ref**: Val**, kbd:HOLE, F.Cu at (350.0, 42.4)
- added Ref**: Val**, kbd:HOLE, F.Cu at (32.3, 139.7)
- moved SW84 321.3 mm to (31.2, 75.4), turned to 270 degrees
- moved SW85 319.0 mm to (351.3, 75.2), turned to 270 degrees
- moved R1 7.64 mm to (30.0, 101.6), turned to 270 degrees
- moved R2 7.62 mm to (33.0, 101.6), turned to 270 degrees
- moved D31 3.81 mm to (132.1, 47.0)
- moved D42 0.89 mm to (222.0, 142.2)
- renumbered J_PIKO_e to J_PIKO_4E1
Connections:
- C1 pad 1: L_VCC3P3V -> L_VCC3P3V_T
- C1 pad 2: GND -> L_GND
- C2 pad 1: VCC3P3V -> VCC3P3V_T
- J1 pad A: GND -> L_GND
- J3 pad 4: GND -> L_GND
- J4 pad 2: GND -> L_GND
- J4 pad 3: GND -> L_GND
- J4 pad 4: L_VCC3P3V -> L_VCC3P3V_T
- J5 pad 4: GND -> L_GND
- J6 pad 4: VCC3P3V -> VCC3P3V_T
- JP1 pad 1: GND -> L_GND
- JP1 pad 3: VCC -> L_VCC5V
- JP2 pad 1: GND -> L_GND
- JP2 pad 3: VCC -> L_VCC5V
- JP3 pad 1: GND -> L_GND
- JP3 pad 3: VCC -> L_VCC5V
- JP_A1 pad 3: VCC -> VCC5V
- JP_A2 pad 3: VCC -> VCC5V
- JP_A3 pad 3: VCC -> VCC5V
- SW84 pad 1: VCC -> L_VCC3P3V
- SW84 pad 2: L_VCC5V -> L_VCC3P3V_T
- SW85 pad 1: VCC -> VCC3P3V
- SW85 pad 2: VCC5V -> VCC3P3V_T
- U1 pad 10: GND -> L_GND
- U2 pad 4: GND -> L_GND
Routing:
- net L_GND: track 0.00 -> 470.7 mm, vias 0 -> 11
- net L_VCC5V: track 694.4 -> 287.9 mm, vias 17 -> 8
- net VCC5V: track 0.00 -> 370.8 mm, vias 0 -> 7
- net GND: track 759.5 -> 413.3 mm, vias 14 -> 4
- net L_G22: track 0.00 -> 150.6 mm, vias 0 -> 1
- net G22: track 0.00 -> 135.5 mm
- net VCC3P3V_T: track 0.00 -> 66.2 mm, vias 0 -> 2
- net G33: track 0.00 -> 52.8 mm
- net L_G33: track 0.00 -> 45.9 mm, vias 0 -> 1
- net L_VCC3P3V_T: track 0.00 -> 40.3 mm
- net L_VCC3P3V: track 121.0 -> 141.3 mm
- net COL_8: track 88.1 -> 74.3 mm
- net L_ROW_4: track 150.9 -> 139.5 mm
- net ROW_5: track 204.0 -> 193.0 mm
- net ROW_0: track 218.0 -> 227.3 mm, vias 0 -> 1
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- removed copper zone on B.Cu, net GND
- removed copper zone on F.Cu, net GND
Other:
- board size 353.7 x 115.6 mm -> 353.1 x 115.6 mm

Commit message: add gerber files.
Parts:
- moved D75 22.6 mm to (293.0, 85.1)
- moved D78 22.6 mm to (320.9, 142.2)
- moved D82 22.6 mm to (320.9, 47.0)
- moved D83 22.6 mm to (320.9, 66.0)
- moved R3 22.6 mm to (308.9, 96.5)
- moved D40 22.6 mm to (183.1, 104.1)
- moved D42 22.6 mm to (199.4, 142.2)
- moved D50 22.6 mm to (206.6, 66.0)
- moved D51 22.6 mm to (216.8, 85.1)
- moved D53 22.6 mm to (230.8, 123.2)
- moved D59 22.6 mm to (249.8, 123.2)
- moved J10 22.6 mm to (154.4, 39.6)
- moved SW37 22.6 mm to (165.2, 38.1)
- moved SW38 22.6 mm to (169.0, 57.1)
- moved SW41 22.6 mm to (192.8, 114.3)
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Routing:
- net L_GND: vias 11 -> 86
- net GND: vias 4 -> 49
- net VCC5V: vias 7 -> 8
- net Net-(D30-Pad2): vias 0 -> 1
- net Net-(D23-Pad2): vias 0 -> 1
- net L_VCC5V: vias 8 -> 9
- net L_G22: vias 1 -> 3
- net L_COL_5: vias 2 -> 3
- net L_COL_3: vias 2 -> 3
- net L_COL_2: vias 2 -> 3
- added copper zone on B.Cu, net GND
- added copper zone on F.Cu, net GND
- added copper zone on B.Cu, net L_GND
- added copper zone on F.Cu, net L_GND
- added copper zone on F.Cu, net Net-(J_PIKO1-Pad3)
- added copper zone on B.Cu, net Net-(J_PIKO1-Pad4)
- added copper zone on F.Cu, net Net-(J_PIKO2-Pad3)
- added copper zone on B.Cu, net Net-(J_PIKO2-Pad4)
- added copper zone on F.Cu, net Net-(J_PIKO3-Pad3)
- added copper zone on B.Cu, net Net-(J_PIKO3-Pad4)
- added copper zone on F.Cu, net Net-(J_PIKO4-Pad3)
- added copper zone on B.Cu, net Net-(J_PIKO4-Pad4)
Other:
- board size 353.1 x 115.6 mm -> 330.5 x 115.6 mm
